Commit message: Make camera static

File: urdf/youbot_camera/camera.urdf.xacro (robot description, xacro)
@@ -9,5 +9,5 @@
 			<xacro:insert_block name="origin" />
       <axis xyz="0 -1 0" />
-      <limit effort="1" velocity="0.1" lower="0" upper="5"/>
+      <limit effort="1" velocity="0.1" lower="0" upper="0"/>
 			<parent link="${parent}" />
 			<child link="${name}_link" />
