Commit message: Set faults

File: urdf/youbot_arm/arm.urdf.xacro (robot description, xacro)
@@ -8,4 +8,14 @@
         <xacro:include filename="$(find youbot_description)/urdf/youbot_arm/limits.urdf.xacro" />
 	<xacro:macro name="youbot_arm" params="parent name *origin">
+		<xacro:property name="fault1" value="0.15" />
+		<xacro:property name="fault2" value="0.09" />
+		<xacro:property name="fault3" value="0.3" />
+		<xacro:property name="fault4" value="0.05" />
+		<xacro:property name="fault5" value="0.3" />
+		<!--<xacro:property name="fault1" value="0.15" />
+		<xacro:property name="fault2" value="0.09" />
+		<xacro:property name="fault3" value="0.2" />
+		<xacro:property name="fault4" value="0.05" />
+		<xacro:property name="fault5" value="0.3" />-->
 		<!-- joint between base_link and arm_0_link -->
 		<joint name="${name}_joint_0" type="fixed" >
@@ -61,5 +71,5 @@
 			</inertial>
 			<visual>
-				<origin xyz="0 0 0" rpy="0 0 0" />
+				<origin xyz="0 0 0" rpy="0 0 ${fault1}" />
 				<geometry>
 					<mesh filename="package://youbot_description/meshes/youbot_arm/arm1.dae" />
@@ -69,5 +79,5 @@
 			<collision>
 				<!--<origin xyz="0 0 -0.003" rpy="0 0 0" />-->
-				<origin xyz="0 0 0" rpy="0 0 0" />
+				<origin xyz="0 0 0" rpy="0 0 ${fault1}" />
 				<geometry>
 					<mesh filename="package://youbot_description/meshes/youbot_arm/arm1_convex.dae" />
@@ -93,5 +103,5 @@
 			</inertial>
 			<visual>
-			<origin xyz="0 -0.032 0.078" rpy="0 0 0" />
+			<origin xyz="0 -0.032 0.078" rpy="${fault2} 0 0" />
 				<geometry>
 					<mesh filename="package://youbot_description/meshes/youbot_arm/arm2.dae" />
@@ -101,5 +111,5 @@
 			<collision>
 				<!--<origin xyz="0.001 -0.041 0.074" rpy="0 0 0" />-->
-				<origin xyz="0 -0.032 0.078" rpy="0 0 0" />
+				<origin xyz="0 -0.032 0.078" rpy="${fault2} 0 0" />
 				<geometry>
 					<mesh filename="package://youbot_description/meshes/youbot_arm/arm2_convex.dae" />
@@ -133,5 +143,5 @@
 			</inertial>
 			<visual>
-				<origin xyz="0.000 0.028 0.079" rpy="0 0 0" />
+				<origin xyz="0.000 0.028 0.079" rpy="${fault3} 0 0" />
 				<geometry>
 					<mesh filename="package://youbot_description/meshes/youbot_arm/arm3.dae" />
@@ -141,5 +151,5 @@
 			<collision>
 				<!--<origin xyz="0.000 0.025 0.067" rpy="0 0 0" />-->
-				<origin xyz="0.000 0.028 0.079" rpy="0 0 0" />
+				<origin xyz="0.000 0.028 0.079" rpy="${fault3} 0 0" />
 				<geometry>
 					<mesh filename="package://youbot_description/meshes/youbot_arm/arm3_convex.dae" />
@@ -165,5 +175,5 @@
 			</inertial>
 			<visual>
-				<origin xyz="0 -0.010 0.029" rpy="0 0 0"/>
+				<origin xyz="0 -0.010 0.029" rpy="${fault4} 0 0"/>
 				<geometry>
 					<mesh filename="package://youbot_description/meshes/youbot_arm/arm4.dae" />
@@ -173,5 +183,5 @@
 			<collision>
 				<!--<origin xyz="0 0 0.026" rpy="0 0 0" />-->
-				<origin xyz="0 -0.010 0.029" rpy="0 0 0"/>
+				<origin xyz="0 -0.010 0.029" rpy="${fault4} 0 ${fault4}"/>
 				<geometry>
 					<mesh filename="package://youbot_description/meshes/youbot_arm/arm4_convex.dae" />
@@ -197,5 +207,5 @@
 			</inertial>
 			<visual>
-				<origin xyz="0.003 0 -0.034" rpy="0 0 0" />
+				<origin xyz="0.003 0 -0.034" rpy="0 0 ${fault5}" />
 				<geometry>
 					<mesh filename="package://youbot_description/meshes/youbot_arm/arm5.dae" />
@@ -204,5 +214,5 @@
 			</visual>
 			<collision>
-				<origin xyz="0.003 0 -0.034" rpy="0 0 0" />
+				<origin xyz="0.003 0 -0.034" rpy="0 0 ${fault5}" />
 				<geometry>
 					<mesh filename="package://youbot_description/meshes/youbot_arm/arm5_convex.dae" />

File: urdf/youbot_gripper/gripper.urdf.xacro (robot description, xacro)
@@ -8,4 +8,5 @@
 	<xacro:include filename="$(find youbot_description)/urdf/youbot_gripper/limits.urdf.xacro" />
 	<xacro:macro name="youbot_gripper" params="parent name *origin">
+		<xacro:property name="fault" value="0.3" />
 		<!-- joint between arm_7_link and sdh_palm_link -->
 		<joint name="${name}_palm_joint" type="fixed" >
@@ -16,10 +17,10 @@
 		<link name="${name}_palm_link">
 			<inertial>
-				<origin xyz="0 0 0" rpy="0 0 0"/>
+				<origin xyz="0 0 0" rpy="0 0 ${fault}"/>
 				<mass value="0.1"/>
 				<inertia ixx="0.01" ixy="0" ixz="0" iyy="0.01" iyz="0" izz="0.01" />
 			</inertial>
 			<visual>
-				<origin xyz="0 0 0" rpy="0 0 0" />
+				<origin xyz="0 0 0" rpy="0 0 ${fault}" />
 				<geometry>
 					<mesh filename="package://youbot_description/meshes/youbot_gripper/palm.dae" />
