Commit message: Fix gripper finger axis

File: urdf/youbot_gripper/gripper.urdf.xacro (robot description, xacro)
@@ -39,5 +39,5 @@
 			<parent link="${name}_palm_link"/>
 			<child link="${name}_finger_link_l"/>
-			<axis xyz="0 -1 0" />
+			<axis xyz="0 1 0" />
 			<dynamics damping="1.0" friction="1.0" />
 			<limit effort="1" velocity="0.1" lower="0" upper="${finger_joint}"/>

Commit message: Fix gripper fingers for no physics mode

File: urdf/youbot_gripper/gripper.urdf.xacro (robot description, xacro)
@@ -36,5 +36,5 @@
 		</link>
 		<joint name="${name}_finger_joint_l" type="prismatic">
-			<origin xyz="0.004 0.008 0.046" rpy="0 0 ${M_PI}" />
+			<origin xyz="-0.002 0.008 0.046" rpy="0 0 ${M_PI}" />
 			<parent link="${name}_palm_link"/>
 			<child link="${name}_finger_link_l"/>
@@ -66,5 +66,5 @@
 		</link>
                <joint name="${name}_finger_joint_r" type="prismatic">
-			<origin xyz="0.004 -0.008 0.046" rpy="0 0 0" />
+			<origin xyz="0.010 -0.008 0.046" rpy="0 0 0" />
 			<parent link="${name}_palm_link"/>
 			<child link="${name}_finger_link_r"/>

File: urdf/youbot_gripper/limits.urdf.xacro (robot description, xacro)
@@ -5,5 +5,5 @@
         <xacro:property name="threshold" value="0.001" />
 	<!-- fingers limits, values are in meters -->
-	<xacro:property name="finger_joint" value="${0.023 / 2.0}" />
+	<xacro:property name="finger_joint" value="${0.035 / 2.0}" />
 	<xacro:property name="finger_joint_soft" value="${(0.023 - threshold) / 2.0}" />
 </robot>

Commit message: Add distance mark

File: urdf/youbot_gripper/gripper.urdf.xacro (robot description, xacro)
@@ -7,4 +7,5 @@
 	<xacro:include filename="$(find youbot_description)/urdf/youbot_gripper/gripper.transmission.xacro" />
 	<xacro:include filename="$(find youbot_description)/urdf/youbot_gripper/limits.urdf.xacro" />
+	<xacro:include filename="$(find youbot_description)/urdf/youbot_gripper/mark.urdf.xacro" />
 	<xacro:macro name="youbot_gripper" params="parent name *origin">
 		<xacro:property name="fault" value="0.3" />
@@ -96,4 +97,7 @@
 			</collision>
 		</link>
+		<xacro:gripper_mark name="mark" parent="${name}_palm_link">
+			<origin xyz="0 0 0.022" rpy="0 0 0" />
+		</xacro:gripper_mark>
 		<!-- extensions -->
 		<xacro:youbot_gripper_gazebo name="${name}" />
